Commit message: backup

File: install/gazebo_tutorial/share/gazebo_tutorial/vision60/vision60_double.urdf (robot description, URDF)
Before this commit: robot ngr, 18 links, 17 joints
Links:
- removed link world
- added link base_link
Joints:
- joint body_joint: origin xyz=0 0 1 rpy=0 0 0 -> xyz=-0.5 0 0.1 rpy=0 0 0; parent world -> base_link

File: install/gazebo_tutorial/share/gazebo_tutorial/vision60/vision60_double.xacro (robot description, xacro)
@@ -1,13 +1,6 @@
 <?xml version="1.0" ?>
-<robot name="ngr" xmlns:xacro="http://www.ros.org/wiki/xacro">
-  <!-- gazebo ros control plugin-->
-  <gazebo reference="world">
-    <plugin name="gazebo_ros_control" filename="libgazebo_ros_control.so">
-      <robotNamespace>/vision60</robotNamespace>
-    </plugin>
-    <static>false</static>
-  </gazebo>
-  <!-- Define parameters -->
-  <!-- Define materials -->
+<robot name="vision60" xmlns:xacro="http://www.ros.org/wiki/xacro">
+  <!--MACROS: pass-->
+  <!--MATERIAL (COLOR)-->
   <material name="gray">
     <color rgba="0.5 0.5 0.5 0.7"/>
@@ -28,10 +21,15 @@
     <color rgba="0.8 0.0 0.2 1.0"/>
   </material>
-  <link name="world"/>
-  <!-- Body -->
-  <!--body joint-->
+  <material name="green">
+    <color rgba = "0.1 1 0.1 1.0"/>
+  </material>
+  <!--BASE LINK-->
+  <link name="base_link">
+  </link>
+  <!--BODY-->
+  <!--BODY JOINT-->
   <joint name="body_joint" type="fixed">
-    <origin xyz="0 0 1" rpy="0 0 0"/>
-    <parent link="world"/>
+    <origin xyz="0.5 0 0.1" rpy="0 0 0"/>
+    <parent link="base_link"/>
     <child link="body"/>
   </joint>
@@ -43,5 +41,5 @@
         <box size="0.88 0.25 0.19"/>
       </geometry>
-      <material name="gray"/>
+      <material name="green"/>
     </visual>
     <inertial>
@@ -57,4 +55,7 @@
     </collision>
   </link>
+  <gazebo reference="body">
+    <material>Gazebo/Green</material>
+  </gazebo>
   <!-- Define our leg macro -->
   <!-- red new legs -->
@@ -82,4 +83,7 @@
     </inertial>
   </link>
+  <gazebo reference="hip0">
+    <material>Gazebo/Red</material>
+  </gazebo>
   <!-- Abduction joint. Joint names are: 8 9 10 11 -->
   <joint name="8" type="revolute">
@@ -111,4 +115,7 @@
     </inertial>
   </link>
+  <gazebo reference="upper0">
+    <material>Gazebo/Blue</material>
+  </gazebo>
   <!-- Hip joint. (Motor to upper leg). Joint names are: 0 2 4 6 -->
   <joint name="0" type="revolute">
@@ -141,4 +148,7 @@
     </inertial>
   </link>
+  <gazebo reference="lower0">
+    <material>Gazebo/Black</material>
+  </gazebo>
   <!-- Knee joint. Joint names are: 1 3 5 7 -->
   <joint name="1" type="revolute">
@@ -178,4 +188,7 @@
     </inertial>
   </link>
+  <gazebo reference="toe0">
+    <material>Gazebo/Gray</material>
+  </gazebo>
   <joint name="jtoe0" type="fixed">
     <parent link="lower0"/>
@@ -204,4 +217,7 @@
     </inertial>
   </link>
+  <gazebo reference="hip1">
+    <material>Gazebo/Purple</material>
+  </gazebo>
   <!-- Abduction joint. Joint names are: 8 9 10 11 -->
   <joint name="9" type="revolute">
@@ -233,4 +249,7 @@
     </inertial>
   </link>
+  <gazebo reference="upper1">
+    <material>Gazebo/Blue</material>
+  </gazebo>
   <!-- Hip joint. (Motor to upper leg). Joint names are: 0 2 4 6 -->
   <joint name="2" type="revolute">
@@ -263,4 +282,7 @@
     </inertial>
   </link>
+  <gazebo reference="lower1">
+    <material>Gazebo/Black</material>
+  </gazebo>
   <!-- Knee joint. Joint names are: 1 3 5 7 -->
   <joint name="3" type="revolute">
@@ -300,4 +322,7 @@
     </inertial>
   </link>
+  <gazebo reference="toe1">
+    <material>Gazebo/Gray</material>
+  </gazebo>
   <joint name="jtoe1" type="fixed">
     <parent link="lower1"/>
@@ -326,4 +351,7 @@
     </inertial>
   </link>
+  <gazebo reference="hip2">
+    <material>Gazebo/Red</material>
+  </gazebo>
   <!-- Abduction joint. Joint names are: 8 9 10 11 -->
   <joint name="10" type="revolute">
@@ -355,4 +383,7 @@
     </inertial>
   </link>
+  <gazebo reference="upper2">
+    <material>Gazebo/Blue</material>
+  </gazebo>
   <!-- Hip joint. (Motor to upper leg). Joint names are: 0 2 4 6 -->
   <joint name="4" type="revolute">
@@ -385,4 +416,7 @@
     </inertial>
   </link>
+  <gazebo reference="lower2">
+    <material>Gazebo/Black</material>
+  </gazebo>
   <!-- Knee joint. Joint names are: 1 3 5 7 -->
   <joint name="5" type="revolute">
@@ -422,4 +456,7 @@
     </inertial>
   </link>
+  <gazebo reference="toe2">
+    <material>Gazebo/Gray</material>
+  </gazebo>
   <joint name="jtoe2" type="fixed">
     <parent link="lower2"/>
@@ -448,4 +485,7 @@
     </inertial>
   </link>
+  <gazebo reference="hip3">
+    <material>Gazebo/Purple</material>
+  </gazebo>
   <!-- Abduction joint. Joint names are: 8 9 10 11 -->
   <joint name="11" type="revolute">
@@ -477,4 +517,7 @@
     </inertial>
   </link>
+  <gazebo reference="upper3">
+    <material>Gazebo/Blue</material>
+  </gazebo>
   <!-- Hip joint. (Motor to upper leg). Joint names are: 0 2 4 6 -->
   <joint name="6" type="revolute">
@@ -507,4 +550,7 @@
     </inertial>
   </link>
+  <gazebo reference="lower3">
+    <material>Gazebo/Black</material>
+  </gazebo>
   <!-- Knee joint. Joint names are: 1 3 5 7 -->
   <joint name="7" type="revolute">
@@ -544,4 +590,7 @@
     </inertial>
   </link>
+  <gazebo reference="toe3">
+    <material>Gazebo/Gray</material>
+  </gazebo>
   <joint name="jtoe3" type="fixed">
     <parent link="lower3"/>
@@ -550,3 +599,5 @@
     <dynamics damping="0.0" friction="0.0"/>
   </joint>
+  <!--Gazebo plugin-->
+  <xacro:include filename="plugin_control.xacro"/>
 </robot>
