Commit message: backup

File: install/gazebo_tutorial/share/gazebo_tutorial/vision60/vision60_double.xacro (robot description, xacro)
@@ -56,5 +56,5 @@
   </link>
   <gazebo reference="body">
-    <material>Gazebo/Green</material>
+    <material>Gazebo/White</material>
   </gazebo>
   <!-- Define our leg macro -->
